Commit message: Initial add of both wheels to robot.xakro

File: src/my_robot/urdf/my_robot.xacro (robot description, xacro)
@@ -5,5 +5,21 @@
         <origin xyz="0 0 0" rpy="0 0 0" />
         <parent link="robot_footprint"/>
-        <child link="chassis" />
+        <child link="chassis"/>
+    </joint>
+    <joint name="left_wheel_hinge" type="continuous">
+        <origin xyz="0 0.15 0" rpy="0 0 0" />
+        <parent link="chassis"/>
+        <child link="left_wheel"/>
+        <axis xyz="0 1 0" rpy="0 0 0"/>
+        <limit effort="10000" velocity="1000"/>
+        <dynamics damping="1.0" friction="1.0"/>
+    </joint>
+    <joint name="right_wheel_hinge" type="continuous">
+        <origin xyz="0 0.15 0" rpy="0 0 0" />
+        <parent link="chassis"/>
+        <child link="left_wheel"/>
+        <axis xyz="0 1 0" rpy="0 0 0"/>
+        <limit effort="10000" velocity="1000"/>
+        <dynamics damping="1.0" friction="1.0"/>
     </joint>
     <link name='chassis'>
@@ -27,5 +43,5 @@
             <origin xyz="0 0 0" rpy=" 0 0 0"/>
             <geometry>
-            <box size=".4 .2 .1"/>
+                <box size=".4 .2 .1"/>
             </geometry>
         </visual>
@@ -33,5 +49,5 @@
             <origin xyz="-0.15 0 -0.05" rpy=" 0 0 0"/>
             <geometry>
-            <sphere radius="0.0499"/>
+                <sphere radius="0.0499"/>
             </geometry>
         </collision>
@@ -39,5 +55,5 @@
             <origin xyz="-0.15 0 -0.05" rpy=" 0 0 0"/>
             <geometry>
-            <sphere radius="0.05"/>
+                <sphere radius="0.05"/>
             </geometry>
         </visual>
@@ -45,5 +61,5 @@
             <origin xyz="0.15 0 -0.05" rpy=" 0 0 0"/>
             <geometry>
-            <sphere radius="0.0499"/>
+                <sphere radius="0.0499"/>
             </geometry>
         </collision>
@@ -51,5 +67,51 @@
             <origin xyz="0.15 0 -0.05" rpy=" 0 0 0"/>
             <geometry>
-            <sphere radius="0.05"/>
+                <sphere radius="0.05"/>
+            </geometry>
+        </visual>
+    </link>
+    <link name='left_wheel'>
+        <pose>0 0 0.1 0 0 0</pose>
+        <inertial>
+            <mass value="5.0"/>
+            <origin xyz="0.0 0 0" rpy=" 0 1.5707 1.5707"/>
+            <inertia
+                ixx="0.1" ixy="0" ixz="0"
+                iyy="0.1" iyz="0" izz="0.1"
+            />
+        </inertial>
+        <collision name='left_wheel_collision'>
+            <origin xyz="0.0 0 0" rpy=" 0 1.5707 1.5707"/>
+            <geometry>
+                <cylinder length="0.05" radius="0.1"/>
+            </geometry>
+        </collision>
+        <visual name='left_wheel_visual'>
+            <origin xyz="0.0 0 0" rpy=" 0 1.5707 1.5707"/>
+            <geometry>
+                <cylinder length="0.05" radius="0.1"/>
+            </geometry>
+        </visual>
+    </link>
+    <link name='right_wheel'>
+        <pose>0 0 0.1 0 0 0</pose>
+        <inertial>
+            <mass value="5.0"/>
+            <origin xyz="0.0 0 0" rpy=" 0 1.5707 1.5707"/>
+            <inertia
+                ixx="0.1" ixy="0" ixz="0"
+                iyy="0.1" iyz="0" izz="0.1"
+            />
+        </inertial>
+        <collision name='right_wheel_collision'>
+            <origin xyz="0.0 0 0" rpy=" 0 1.5707 1.5707"/>
+            <geometry>
+                <cylinder length="0.05" radius="0.1"/>
+            </geometry>
+        </collision>
+        <visual name='right_wheel_visual'>
+            <origin xyz="0.0 0 0" rpy=" 0 1.5707 1.5707"/>
+            <geometry>
+                <cylinder length="0.05" radius="0.1"/>
             </geometry>
         </visual>

Commit message: Correct the y=-0.15 for the right wheel joint

File: src/my_robot/urdf/my_robot.xacro (robot description, xacro)
@@ -16,7 +16,7 @@
     </joint>
     <joint name="right_wheel_hinge" type="continuous">
-        <origin xyz="0 0.15 0" rpy="0 0 0" />
+        <origin xyz="0 -0.15 0" rpy="0 0 0" />
         <parent link="chassis"/>
-        <child link="left_wheel"/>
+        <child link="right_wheel"/>
         <axis xyz="0 1 0" rpy="0 0 0"/>
         <limit effort="10000" velocity="1000"/>

Commit message: Add camera sensor to the robot udtf

File: src/my_robot/urdf/my_robot.xacro (robot description, xacro)
@@ -22,4 +22,10 @@
         <limit effort="10000" velocity="1000"/>
         <dynamics damping="1.0" friction="1.0"/>
+    </joint>
+    <joint name="camera_joint" type="fixed">
+        <origin xyz="0.2 0 0" rpy="0 0 0" />
+        <parent link="chassis"/>
+        <child link="camera"/>
+        <axis xyz="0 1 0" rpy="0 0 0"/>
     </joint>
     <link name='chassis'>
@@ -117,3 +123,26 @@
         </visual>
     </link>
+    <link name='camera'>
+        <pose>0 0 0.1 0 0 0</pose>
+        <inertial>
+            <mass value="0.1"/>
+            <origin xyz="0.0 0 0" rpy=" 0 0 0"/>
+            <inertia
+                ixx="1e-6" ixy="0" ixz="0"
+                iyy="1e-6" iyz="0" izz="1e-6"
+            />
+        </inertial>
+        <collision name='camera_collision'>
+            <origin xyz="0.0 0 0" rpy=" 0 1.5707 1.5707"/>
+            <geometry>
+                <box size="0.05 0.05 0.05"/>
+            </geometry>
+        </collision>
+        <visual name='camera_visual'>
+            <origin xyz="0.0 0 0" rpy=" 0 1.5707 1.5707"/>
+            <geometry>
+                <box size="0.05 0.05 0.05"/>
+            </geometry>
+        </visual>
+    </link>
 </robot>

Commit message: Add the link and joint for the lidar in the urft file

File: src/my_robot/urdf/my_robot.xacro (robot description, xacro)
@@ -27,4 +27,10 @@
         <parent link="chassis"/>
         <child link="camera"/>
+        <axis xyz="0 1 0" rpy="0 0 0"/>
+    </joint>
+    <joint name="hokuyo_joint" type="fixed">
+        <origin xyz="0.15 0 0.1" rpy="0 0 0" />
+        <parent link="chassis"/>
+        <child link="hokuyo"/>
         <axis xyz="0 1 0" rpy="0 0 0"/>
     </joint>
@@ -146,3 +152,26 @@
         </visual>
     </link>
+    <link name='hokuyo'>
+        <pose>0 0 0.1 0 0 0</pose>
+        <inertial>
+            <mass value="1e-5"/>
+            <origin xyz="0 0 0" rpy=" 0 0 0"/>
+            <inertia
+                ixx="1e-6" ixy="0" ixz="0"
+                iyy="1e-6" iyz="0" izz="1e-6"
+            />
+        </inertial>
+        <collision name='hokuyo_collision'>
+            <origin xyz="0 0 0" rpy=" 0 0 0"/>
+            <geometry>
+                <box size="0.1 0.1 0.1"/>
+            </geometry>
+        </collision>
+        <visual name='hokuyo_visual'>
+            <origin xyz="0 0 0" rpy=" 0 0 0"/>
+            <geometry>
+                <mesh filename="package://robotics/src/my_robot/meshes/hokuyo.dae"/>
+            </geometry>
+        </visual>
+    </link>
 </robot>

Commit message: Correct path for tlidar shape file

File: src/my_robot/urdf/my_robot.xacro (robot description, xacro)
@@ -171,5 +171,5 @@
             <origin xyz="0 0 0" rpy=" 0 0 0"/>
             <geometry>
-                <mesh filename="package://robotics/src/my_robot/meshes/hokuyo.dae"/>
+                <mesh filename="package://my_robot/meshes/hokuyo.dae"/>
             </geometry>
         </visual>

Commit message: Small syntax corrections on robot.xacro

File: src/my_robot/urdf/my_robot.xacro (robot description, xacro)
@@ -156,5 +156,5 @@
         <inertial>
             <mass value="1e-5"/>
-            <origin xyz="0 0 0" rpy=" 0 0 0"/>
+            <origin xyz="0 0 0" rpy="0 0 0"/>
             <inertia
                 ixx="1e-6" ixy="0" ixz="0"
@@ -163,5 +163,5 @@
         </inertial>
         <collision name='hokuyo_collision'>
-            <origin xyz="0 0 0" rpy=" 0 0 0"/>
+            <origin xyz="0 0 0" rpy="0 0 0"/>
             <geometry>
                 <box size="0.1 0.1 0.1"/>
@@ -169,5 +169,5 @@
         </collision>
         <visual name='hokuyo_visual'>
-            <origin xyz="0 0 0" rpy=" 0 0 0"/>
+            <origin xyz="0 0 0" rpy="0 0 0"/>
             <geometry>
                 <mesh filename="package://my_robot/meshes/hokuyo.dae"/>

Commit message: Adding color feature to my_robot.xacro

File: src/my_robot/urdf/my_robot.xacro (robot description, xacro)
@@ -57,4 +57,5 @@
             <geometry>
                 <box size=".4 .2 .1"/>
+                <material name="blue"/>
             </geometry>
         </visual>
@@ -104,4 +105,5 @@
             <geometry>
                 <cylinder length="0.05" radius="0.1"/>
+                <material name="green"/>
             </geometry>
         </visual>
@@ -127,4 +129,5 @@
             <geometry>
                 <cylinder length="0.05" radius="0.1"/>
+                <material name="green"/>
             </geometry>
         </visual>
@@ -150,4 +153,5 @@
             <geometry>
                 <box size="0.05 0.05 0.05"/>
+                <material name="red"/>
             </geometry>
         </visual>

Commit message: Added color to my_robot.xacro

File: src/my_robot/urdf/my_robot.xacro (robot description, xacro)
@@ -57,6 +57,8 @@
             <geometry>
                 <box size=".4 .2 .1"/>
-                <material name="blue"/>
             </geometry>
+            <material name="">
+                <color rgba="0 0 0.8 1"/>
+            </material>
         </visual>
         <collision name='back_caster_collision'>
@@ -89,5 +91,5 @@
         <inertial>
             <mass value="5.0"/>
-            <origin xyz="0.0 0 0" rpy=" 0 1.5707 1.5707"/>
+            <origin xyz="0 0 0" rpy=" 0 1.5707 1.5707"/>
             <inertia
                 ixx="0.1" ixy="0" ixz="0"
@@ -96,5 +98,5 @@
         </inertial>
         <collision name='left_wheel_collision'>
-            <origin xyz="0.0 0 0" rpy=" 0 1.5707 1.5707"/>
+            <origin xyz="0 0 0" rpy=" 0 1.5707 1.5707"/>
             <geometry>
                 <cylinder length="0.05" radius="0.1"/>
@@ -102,9 +104,11 @@
         </collision>
         <visual name='left_wheel_visual'>
-            <origin xyz="0.0 0 0" rpy=" 0 1.5707 1.5707"/>
+            <origin xyz="0 0 0" rpy=" 0 1.5707 1.5707"/>
             <geometry>
                 <cylinder length="0.05" radius="0.1"/>
-                <material name="green"/>
             </geometry>
+            <material name="">
+                <color rgba="0 1 0 1"/>
+            </material>
         </visual>
     </link>
@@ -113,5 +117,5 @@
         <inertial>
             <mass value="5.0"/>
-            <origin xyz="0.0 0 0" rpy=" 0 1.5707 1.5707"/>
+            <origin xyz="0 0 0" rpy=" 0 1.5707 1.5707"/>
             <inertia
                 ixx="0.1" ixy="0" ixz="0"
@@ -120,5 +124,5 @@
         </inertial>
         <collision name='right_wheel_collision'>
-            <origin xyz="0.0 0 0" rpy=" 0 1.5707 1.5707"/>
+            <origin xyz="0 0 0" rpy=" 0 1.5707 1.5707"/>
             <geometry>
                 <cylinder length="0.05" radius="0.1"/>
@@ -126,9 +130,11 @@
         </collision>
         <visual name='right_wheel_visual'>
-            <origin xyz="0.0 0 0" rpy=" 0 1.5707 1.5707"/>
+            <origin xyz="0 0 0" rpy=" 0 1.5707 1.5707"/>
             <geometry>
                 <cylinder length="0.05" radius="0.1"/>
-                <material name="green"/>
             </geometry>
+            <material name="">
+                <color rgba="0 1 0 1"/>
+            </material>
         </visual>
     </link>
@@ -137,5 +143,5 @@
         <inertial>
             <mass value="0.1"/>
-            <origin xyz="0.0 0 0" rpy=" 0 0 0"/>
+            <origin xyz="0 0 0" rpy=" 0 0 0"/>
             <inertia
                 ixx="1e-6" ixy="0" ixz="0"
@@ -144,5 +150,5 @@
         </inertial>
         <collision name='camera_collision'>
-            <origin xyz="0.0 0 0" rpy=" 0 1.5707 1.5707"/>
+            <origin xyz="0 0 0" rpy=" 0 1.5707 1.5707"/>
             <geometry>
                 <box size="0.05 0.05 0.05"/>
@@ -150,9 +156,11 @@
         </collision>
         <visual name='camera_visual'>
-            <origin xyz="0.0 0 0" rpy=" 0 1.5707 1.5707"/>
+            <origin xyz="0 0 0" rpy=" 0 1.5707 1.5707"/>
             <geometry>
                 <box size="0.05 0.05 0.05"/>
-                <material name="red"/>
             </geometry>
+            <material name="">
+                <color rgba="1 0 0 1"/>
+            </material>
         </visual>
     </link>
